File: Schematics/G7 Senior Design V2/G7 Senior Design V2.kicad_sch (KiCad schematic)
At the start: 26 parts, among them IC1 TPS62122DRVR, IC3 CP2102N-A02-GQFN28, J1 87583-2010RLF, J2 PJ-051AH, Q1 SS8050-G, Q2 SS8050-G, U1 ESP32-WROOM-32-N4, U2 DWM1000

Commit message: Added Changes from Last Meeting
Parts:
- removed C3-0.1uF3: CC0805KRX7R9BB104, CC0805N_YAG, symbol 2024-09-06_13-28-08:CC0805KRX7R9BB104
- removed R3-10K2: ERJ-6GEYJ103V, SD V2 USB to UART Components:RC0805N_PAN, symbol 2024-09-06_12-42-36:ERJ-6GEYJ103V
- added C14-0.1uF1, C14-0.1uF3, C15-0.1uF4, C3-0.1uF4, C9-0.1uF2: CC0805KRX7R9BB104, SD V2 ESP32 Components:CC0805N_YAG, symbol 2024-09-06_13-28-08:CC0805KRX7R9BB104
- added C3-22uF2: LMK212BJ226MG-T, SD V2 ESP32 Components:CAP_LMK212AB7106MG-T_TAY, symbol 2024-09-06_13-19-00:LMK212BJ226MG-T
- added LED1, LED2, LED3, LED4, LED5: HSMW-C170-U0000, SD V2 DW1000 Components:LEDC2012X90N, symbol HSMW-C170-U0000:HSMW-C170-U0000
- added R11-10K2, R3-10K5, R3-10K6: ERJ-6GEYJ103V, SD V2 USB to UART Components:RC0805N_PAN, symbol 2024-09-06_12-42-36:ERJ-6GEYJ103V
- added R3-0-Ohms1: RMCF0805ZT0R00, STA_RMCF0805_STP, symbol 2024-09-09_17-13-58:RMCF0805ZT0R00
- added R3-1K2, R3-1K3, R3-1K4, R3-1K5: RG2012P-105-B-T5, SD V2 USB to UART Components:RES_1220_SUS, symbol 2024-09-04_21-57-04:RG2012P-105-B-T5
- added S1, S2: PTS_647_SN50_SMTR2_LFS, SD V2 ESP32 Components:SW_PTS_647_SN50_SMTR2_LFS, symbol PTS_647_SN50_SMTR2_LFS:PTS_647_SN50_SMTR2_LFS
- C21-22uF1: renamed from C3-22uF1; footprint CAP_LMK212AB7106MG-T_TAY -> SD V2 ESP32 Components:CAP_LMK212AB7106MG-T_TAY
- C22-0.1uF2: renamed from C3-0.1uF2; footprint CC0805N_YAG -> SD V2 ESP32 Components:CC0805N_YAG
- Q1, Q2: footprint TRAN_SS8050-G_CIP -> SD V2 USB to UART Components:TRAN_SS8050-G_CIP
- renumbered C3-0.1uF1 to C19-0.1uF1, C3-4.7uF1 to C20-4.7uF1, R3-10K3 to R21-10K3, R3-10K4 to R22-10K4, R3-10K1 to R23-10K1, R3-1K1 to R24-1K1, R3-22.1K1 to R25-22.1K1, R3-47.5K1 to R26-47.5K1
Connections:
- net GND: now also C14-0.1uF1.1, C14-0.1uF3.1, C15-0.1uF4.1, C3-0.1uF4.2, C3-22uF2.2, C9-0.1uF2.1, LED1.1 (K), LED2.1 (K), LED3.1 (K), LED4.1 (K), LED5.1 (K), R3-10K6.2, S1.1, S2.1
- net at C19-0.1uF1.1, C20-4.7uF1.1, C21-22uF1.1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: now also C3-0.1uF4.1, C3-22uF2.1, R11-10K2.1, R3-0-Ohms1.2, R3-10K5.1; no longer C1.1, C2.1, IC1.2 (VOUT), L1.1, R1.2
- net EN: now reaches Q1.3, U1.3 (EN)
- net EN: now also C14-0.1uF1.2, C9-0.1uF2.2, R11-10K2.2, S2.3
- net at U1.12 (IO27): now also R3-1K5.1
- net IO0: now reaches Q2.3, U1.25 (IO0)
- net IO0: now also C14-0.1uF3.2, C15-0.1uF4.2, R3-10K5.2, S1.3
- net at U1.6 (IO34): now also U2.22 (IRQ/GPIO8), R3-10K6.1
- net at U1.8 (IO32): now also R3-1K4.1
- net at U1.9 (IO33): now also R3-1K3.1
- net at U2.1 (EXTON): now also R3-1K3.2
- net at U2.12 (GPIO3/TXLED): now also LED5.2 (A)
- net at U2.13 (GPIO2/RXLED): now also LED1.2 (A)
- net at U2.14 (GPIO1/SFDLED): now also LED2.2 (A)
- net at U2.15 (GPIO0/RXOKLED): now also LED3.2 (A)
- net at U2.2 (WAKEUP): now also R3-1K4.2
- net at U2.3 (RSTN): now also R3-1K5.2
- new net: C1.1, C2.1, IC1.2 (VOUT), L1.1, R1.2, R3-0-Ohms1.1, R3-1K2.1
- new net: LED4.2 (A), R3-1K2.2
Other:
- note added: "3V3"
- note removed: "Vout"
