File: Schematics/G7 Senior Design V2/G7 Senior Design V2.kicad_sch (KiCad schematic)
At the start: 43 parts, among them IC1 TPS62122DRVR, IC3 CP2102N-A02-GQFN28, J1 87583-2010RLF, J2 PJ-051AH, Q1 SS8050-G, Q2 SS8050-G, U1 ESP32-WROOM-32-N4, U2 DWM1000

Commit message: First Version to be Ordered from JLCPCB
Associated schematic with first Gerber file to be sent out to JLCPCB to be fabricated.
Parts:
- removed C1: CC0805JRNPO9BN220, SD V2 Voltage Regulator Components:Cff-22pF CAP_CC0805_YAG, symbol 2024-08-05_16-00-45:CC0805JRNPO9BN220
- removed C2: 08056D475MAT2A, SD V2 Voltage Regulator Components:Cout-4.7uF CAP_0805N_AVX, symbol 2024-08-05_16-10-25:08056D475MAT2A
- removed Cin-4.7uF1: VJ0805A4R7BXXPW1BC, SD V2 Voltage Regulator Components:Cin-CAP_VJ0805_VIS, symbol 2024-08-05_15-15-11:VJ0805A4R7BXXPW1BC
- removed IC1: TPS62122DRVR, SD V2 Voltage Regulator Components:SON65P200X200X80-7N, symbol TPS62122DRVR:TPS62122DRVR
- removed L1: LPS3015-183MRC, SD V2 Voltage Regulator Components:L1-18uH LPS3015183MRC, symbol LPS3015-183MRC:LPS3015-183MRC
- removed LED4: HSMW-C170-U0000, SD V2 DW1000 Components:LEDC2012X90N, symbol HSMW-C170-U0000:HSMW-C170-U0000
- removed R1: RC0805FR-07560KL, SD V2 Voltage Regulator Components:R1-560K RC0805N_YAG, symbol 2024-08-05_15-40-12:RC0805FR-07560KL
- removed R2: CRGCQ0805F180K, SD V2 Voltage Regulator Components:R2-180K RESC2012X65N, symbol CRGCQ0805F180K:CRGCQ0805F180K
- removed R24-1K1, R3-1K2: RG2012P-105-B-T5, SD V2 USB to UART Components:RES_1220_SUS, symbol 2024-09-04_21-57-04:RG2012P-105-B-T5
- added C1: 22uF, SD V2 ESP32 Components:CAP_LMK212AB7106MG-T_TAY, symbol 2024-09-06_13-19-002:LMK212BJ226MG-T
- added C3-22uF1: LMK212BJ226MG-T, SD V2 ESP32 Components:CAP_LMK212AB7106MG-T_TAY, symbol 2024-09-06_13-19-002:LMK212BJ226MG-T
- added J3, J4: PPTC191LFBN-RC, CONN19_PPTC191LFBN-RC_SUL, symbol 2024-09-12_12-58-59:PPTC191LFBN-RC
- added LED1: RED, SD V2 DW1000 Components:LEDC2012X90N, symbol HSMW-C170-U0000:HSMW-C170-U0000
- added R2, R24: 2K, SD V2 USB to UART Components:RESC2012X60N, symbol RC0805JR-072KL:RC0805JR-072KL
- added R4, R5, R6, R7: CRGCQ0805J470R, SD V2 DW1000 Components:RESC2012X65N, symbol CRGCQ0805J470R:CRGCQ0805J470R
- added U3: AMS1117-3.3, SD V2 Voltage Regulator Components:SOT229P700X180-4N, symbol AMS1117-3.3:AMS1117-3.3
- C14: renamed from C14-0.1uF1; value CC0805KRX7R9BB104 -> 0.1uF
- C15: renamed from C15-0.1uF4; value CC0805KRX7R9BB104 -> C15
- C19: renamed from C19-0.1uF1; value GRM219C80J475KE19D -> 0.1uF
- C20: renamed from C20-4.7uF1; value GRM219C80J475KE19D -> 4.7uF
- C21: renamed from C21-22uF1; value LMK212BJ226MG-T -> 22uF
- C22: renamed from C22-0.1uF2; value CC0805KRX7R9BB104 -> 0.1uF
- C3: renamed from C3-0.1uF4; value CC0805KRX7R9BB104 -> C6
- C31: renamed from C3-22uF2; value LMK212BJ226MG-T -> C5
- D1: renamed from LED5; value HSMW-C170-U0000 -> LD1
- D2: renamed from LED1; value HSMW-C170-U0000 -> LD2
- D3: renamed from LED2; value HSMW-C170-U0000 -> LD3
- D4: renamed from LED3; value HSMW-C170-U0000 -> LD4
- IC3: value CP2102N-A02-GQFN28 -> UART
- J1: value 87583-2010RLF -> USB
- J2: value PJ-051AH -> JCK
- Q1: value SS8050-G -> T1
- Q2: value SS8050-G -> T2
- R0-1: renamed from R3-0-Ohms1; value RMCF0805ZT0R00 -> 0K; footprint STA_RMCF0805_STP -> SD V2 Voltage Regulator Components:STA_RMCF0805_STP
- R11: renamed from R11-10K2; value ERJ-6GEYJ103V -> R11
- R15-1: renamed from R3-10K6; value ERJ-6GEYJ103V -> 10K
- R21: renamed from R21-10K3; value ERJ-6GEYJ103V -> 10K
- R22: renamed from R22-10K4; value ERJ-6GEYJ103V -> 10K
- R23: renamed from R23-10K1; value ERJ-6GEYJ103V -> 10K
- R25: renamed from R25-22.1K1; value RMCF0805FT22K1 -> 22.1K
- R26: renamed from R26-47.5K1; value RMCF0805FT47K5 -> 47.5K
- R31: renamed from R3-1K5; value RG2012P-105-B-T5 -> RD1
- R32: renamed from R3-1K4; value RG2012P-105-B-T5 -> RD2
- R33: renamed from R3-1K3; value RG2012P-105-B-T5 -> RD3
- R34: renamed from R3-10K5; value ERJ-6GEYJ103V -> 10K
- S1: value PTS_647_SN50_SMTR2_LFS -> S1
- S2: value PTS_647_SN50_SMTR2_LFS -> S2
Connections:
- net EN: now also U1.14 (IO12), J3.7
- net GND: now also C1.1, C3-22uF1.2, LED1.1 (K), U3.1 (GND/ADJ); no longer J1.S1 (SHIELD), J1.S2 (SHIELD__1), J2.S1 (SHIELD), J2.S2 (SHIELD__1)
- net at R0-1.1: now also C3-22uF1.1, U3.2 (VOUT)
- net at U1.10 (IO25): now also J3.4
- net at U1.11 (IO26): now also J3.5
- net at U1.13 (IO14): now also J3.6
- net at U1.16 (IO13): now also J3.8
- net at U1.17 (SD2): now also J3.9
- net at U1.18 (SD3): now also J3.10
- net at U1.19 (CMD): now also J4.1
- net at C19.1, C20.1, C21.1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: now also R24.1
- net at U1.20 (CLK): now also J4.2
- net at U1.21 (SD0): now also J3.11
- net at U1.22 (SD1): now also J3.12
- net at U1.23 (IO15): now also J3.13
- net at U1.24 (IO2): now also J3.19
- net at U1.27 (IO16): now also J3.18
- net at U1.28 (IO17): now also J3.17
- net at U1.29 (IO5): now also J3.16
- net at U1.33 (IO21): now also J3.15
- net at U1.36 (IO22): now also J3.14
- net at U1.4 (SENSOR_VP): now also J3.1
- net at U1.5 (SENSOR_VN): now also J3.2
- net at U1.7 (IO35): now also J3.3
- net at D3.2 (A): now also R7.2; no longer U2.14 (GPIO1/SFDLED)
- net at IC3.9 (RSTB): now also R24.2
- net at D4.2 (A): now also R6.2; no longer U2.15 (GPIO0/RXOKLED)
- net at U2.13 (GPIO2/RXLED): now also R4.1; no longer D2.2 (A)
- net at J2.1: now also C1.2, R2.1, U3.3 (VIN)
- net at D1.2 (A): now also R5.2; no longer U2.12 (GPIO3/TXLED)
- net at U2.10 (GPIO5/EXTTXE/SPIPOL): now also J4.5
- net at U2.11 (GPIO4/EXTPA): now also J4.6
- net at U2.4 (GPIO7): now also J4.3
- net at U2.9 (GPIO6/EXTRXE/SPIPHA): now also J4.4
- new net: LED1.2 (A), R2.2
- new net: D2.2 (A), R4.2
- new net: R7.1, U2.14 (GPIO1/SFDLED)
- new net: R5.1, U2.12 (GPIO3/TXLED)
- new net: R6.1, U2.15 (GPIO0/RXOKLED)
- no-connect marks 0 -> 19
Other:
- note added: "+5V"
- note removed: "+12V"
- note removed: "12V to 3V Regulator"
- moved on the sheet: D1, D2, D3, D4

Commit message: Updated Gerber and BOM 13 SEP 24
Parts:
- removed C19: 0.1uF, SD V2 USB to UART Components:CAPC2012X95N, symbol GRM219C80J475KE19D:GRM219C80J475KE19D
- removed R31: RD1, SD V2 USB to UART Components:RES_1220_SUS, symbol 2024-09-04_21-57-04:RG2012P-105-B-T5
- removed R32: RD2, SD V2 USB to UART Components:RES_1220_SUS, symbol 2024-09-04_21-57-04:RG2012P-105-B-T5
- removed R33: RD3, SD V2 USB to UART Components:RES_1220_SUS, symbol 2024-09-04_21-57-04:RG2012P-105-B-T5
- added C19: 0.1uF, SD V2 USB to UART Components:CAPC2012X145N, symbol VJ0805Y104KXABE31:VJ0805Y104KXABE31
- added R31, R32, R33: 1K, SD V2 DW1000 Components:RC0805N_YAG, symbol 2024-09-13_12-09-25:RC0805FR-071KL
- J3, J4: footprint CONN19_PPTC191LFBN-RC_SUL -> SD V2 ESP32 Components:CONN19_PPTC191LFBN-RC_SUL
Connections:
- net GND: now also C19.2
- net at U1.9 (IO33): now also R33.1
- net at U2.1 (EXTON): now also R33.2
- net at U1.12 (IO27): now also R31.1
- net at C20.1, C21.1, C22.1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: now also C19.1
- net at U1.8 (IO32): now also R32.1
- net at U2.3 (RSTN): now also R31.2
- net at U2.2 (WAKEUP): now also R32.2

Commit message: ChairGuru V1.1
Updated Changes According to Doc as of 06 OCT 24.
Parts:
- added D5, D6: LD1, SD V2 DW1000 Components:LEDC2012X90N, symbol HSMW-C170-U0000:HSMW-C170-U0000
- added R1, R3: CRGCQ0805J470R, SD V2 DW1000 Components:RESC2012X65N, symbol CRGCQ0805J470R:CRGCQ0805J470R
- renumbered C3-22uF1 to C3-1
Connections:
- net EN: no longer J3.7, U1.14 (IO12)
- net GND: now also J4.10, J4.11, J4.12, J4.13, J4.14, J4.15, J4.16, J4.17, J4.18, J4.19, J4.7, J4.8, J4.9, D5.1 (K), D6.1 (K)
- net at J1.01 (VCC), R25.1: now also R1.1
- net at J3.19, U1.24 (IO2): now also R3.1
- net at U1.34 (RXD0): now also IC3.26 (TXD); no longer IC3.25 (RXD)
- net at U1.35 (TXD0): now also IC3.25 (RXD); no longer IC3.26 (TXD)
- new net: J3.7, U1.14 (IO12)
- new net: D5.2 (A), R1.2
- new net: D6.2 (A), R3.2
Other:
- moved on the sheet: C14

Commit message: ChairGuru V2.0.1
11 OCT 24 Updates
Connections:
- net GND: now also J4.2, J4.3, J4.4, J4.6; no longer J4.11, J4.14, J4.17, J4.8
- net at U1.20 (CLK): now also J4.5; no longer J4.2
- net at U2.4 (GPIO7): now also J4.8; no longer J4.3
- net at U2.9 (GPIO6/EXTRXE/SPIPHA): now also J4.11; no longer J4.4
- net at U2.10 (GPIO5/EXTTXE/SPIPOL): now also J4.14; no longer J4.5
- net at U2.11 (GPIO4/EXTPA): now also J4.17; no longer J4.6
