File: Schematics/G7 Senior Design V2/_autosave-G7 Senior Design V2.kicad_sch (KiCad schematic)
At the start: 43 parts, among them IC1 TPS62122DRVR, IC3 CP2102N-A02-GQFN28, J1 87583-2010RLF, J2 PJ-051AH, Q1 SS8050-G, Q2 SS8050-G, U1 ESP32-WROOM-32-N4, U2 DWM1000

Commit message: labels adjusted
Parts:
- C1: value CC0805JRNPO9BN220 -> C1
- C14: renamed from C14-0.1uF1; value CC0805KRX7R9BB104 -> C14
- C15: renamed from C15-0.1uF4; value CC0805KRX7R9BB104 -> C15
- C19: renamed from C19-0.1uF1; value GRM219C80J475KE19D -> C19
- C2: value 08056D475MAT2A -> C2
- C20: renamed from C20-4.7uF1; value GRM219C80J475KE19D -> C20
- C21: renamed from C21-22uF1; value LMK212BJ226MG-T -> C21
- C22-0.1uF2: value CC0805KRX7R9BB104 -> C22
- C3: renamed from C3-0.1uF4; value CC0805KRX7R9BB104 -> C6
- C31: renamed from C3-22uF2; value LMK212BJ226MG-T -> C5
- Cin1: renamed from Cin-4.7uF1; value VJ0805A4R7BXXPW1BC -> Cin
- IC1: value TPS62122DRVR -> REG
- IC3: value CP2102N-A02-GQFN28 -> UART
- J1: value 87583-2010RLF -> USB
- J2: value PJ-051AH -> JCK
- L1: value LPS3015-183MRC -> L1
- LED1: value HSMW-C170-U0000 -> LD2
- LED2: value HSMW-C170-U0000 -> LD3
- LED3: value HSMW-C170-U0000 -> LD4
- LED4: value HSMW-C170-U0000 -> LED1
- LED5: value HSMW-C170-U0000 -> LD5
- Q1: value SS8050-G -> T1
- Q2: value SS8050-G -> T2
- R1: value RC0805FR-07560KL -> R1
- R11: renamed from R11-10K2; value ERJ-6GEYJ103V -> R11
- R2: value CRGCQ0805F180K -> R2
- R21: renamed from R21-10K3; value ERJ-6GEYJ103V -> R21
- R22: renamed from R22-10K4; value ERJ-6GEYJ103V -> R22
- R23: renamed from R23-10K1; value ERJ-6GEYJ103V -> R23
- R24: renamed from R24-1K1; value RG2012P-105-B-T5 -> R24
- R25: renamed from R25-22.1K1; value RMCF0805FT22K1 -> R25
- R26: renamed from R26-47.5K1; value RMCF0805FT47K5 -> R26
- R3: renamed from R3-0-Ohms1; value RMCF0805ZT0R00 -> 0k
- R31: renamed from R3-1K5; value RG2012P-105-B-T5 -> RD1
- R32: renamed from R3-1K4; value RG2012P-105-B-T5 -> RD2
- R33: renamed from R3-1K3; value RG2012P-105-B-T5 -> RD3
- R34: renamed from R3-10K5; value ERJ-6GEYJ103V -> R3
- R35: renamed from R3-10K6; value ERJ-6GEYJ103V -> R31
- R36: renamed from R3-1K2; value RG2012P-105-B-T5 -> R3
- S1: value PTS_647_SN50_SMTR2_LFS -> S1
- S2: value PTS_647_SN50_SMTR2_LFS -> S3
