File: Schematics/G7 Senior Design V2/_autosave-G7 Senior Design V2.kicad_pcb (KiCad board)
At the start: 2 copper layers, 100 x 100 mm, 45 parts, among them IC3 UART, J1 USB, J2 JCK, J3 PPTC191LFBN-RC, J4 PPTC191LFBN-RC, Q1 T1, Q2 T2, U1 ESP32-WROOM-32-N4, U2 DWM1000, U3 AMS1117-3.3

Commit message: added logos and final review, going to order
Parts:
- added G***: LOGO, SD V2 ESP32 Components:UCF Logo 2, F.Cu at (138.5, 102.5)
